File: PCB_EMA/EMA_3/board.brd (EAGLE design)
At the start: 120 x 120 mm, 28 parts

Commit message: added PCBS and EAGLE filfes
Parts:
- added ., LORA: (no value), pinhead:1X08
- added BUS_B: (no value), con-ptr500:AK500/4-H
- added JP10, JP11, JP12, JP13, JP14, JP15, JP16, JP17, JP18, JP19, JP20, JP4, JP5, JP6, JP7, JP8, JP9: (no value), pinhead:1X01
- added VBAT_B: (no value), con-ptr500:AK500/2-H
- BUS: value RJ45-6L-B -> (none); device con-tycoelectronics:RJ45-NO-SHIELD -> pinhead:1X04
- DISPLAY: device pinhead:1X06 -> pinhead:1X04
- moved DISPLAY 86.3 mm to (108.7, 93.4), turned to 0 degrees
- moved C5 34.0 mm to (65.2, 26.0), turned to 270 degrees
- moved SIM800L 26.6 mm to (43.7, 31.2)
- moved _ 26.6 mm to (41.2, 53.2)
- moved LEDS 10.5 mm to (9.20, 93.5)
- moved BUS 4.89 mm to (108.7, 102.8)
- moved R1 2.12 mm to (25.8, 96.5)
- moved R2 1.80 mm to (17.3, 96.4)
- moved R3 1.50 mm to (27.3, 106.3)
Connections:
- removed net N$12: BOARD1.D12, JP2.12
- removed net N$17: BOARD1.3V3, JP1.15
- removed net N$28: BOARD1.D15, JP1.13
- new net 3V3: ..3, BOARD1.3V3, JP1.15
- new net DIO0: ..5, BOARD1.D15, JP1.13
- new net DMISO: BOARD1.D12, JP2.12, LORA.4
- new net N$27: LORA.6
- new net N$29: LORA.7
- net DCS: now also JP13.1, JP14.1, LORA.2; no longer DISPLAY.6
- net DMOSI: now also LORA.3; no longer DISPLAY.4
- net DRST: now also ..4; no longer DISPLAY.5
- net DSCK: now also LORA.5; no longer DISPLAY.3
- net GND: now also ..1, ..2, BUS.3, BUS_B.3, DISPLAY.4, JP15.1, JP16.1, JP17.1, JP18.1, JP19.1, JP20.1, LORA.1, LORA.8, VBAT_B.2; no longer BUS.7, DISPLAY.1
- net MISO: now also JP11.1, JP12.1
- net SCL: now also BUS.2, BUS_B.2, DISPLAY.2, JP10.1, JP9.1; no longer BUS.6
- net SDA: now also BUS.1, BUS_B.1, DISPLAY.1, JP7.1, JP8.1; no longer BUS.5
- net VCC: now also BUS.4, BUS_B.4, DISPLAY.3, JP4.1, JP5.1, JP6.1; no longer BUS.8, DISPLAY.2
- net VIN: now also VBAT_B.1
Routing:
- net 3V3: track 0.00 -> 113.9 mm
- net DIO0: track 0.00 -> 107.2 mm
- net DMISO: track 0.00 -> 52.8 mm
- net SCL: track 163.8 -> 212.7 mm
- net SDA: track 159.1 -> 205.5 mm
- net VCC: track 371.1 -> 333.3 mm
- net VIN: track 79.3 -> 113.4 mm
- net DRST: track 79.0 -> 111.7 mm
- net DMOSI: track 28.6 -> 57.3 mm
- net DSCK: track 29.7 -> 48.4 mm
- net DCS: track 100.8 -> 116.7 mm
- net N$12: track 12.4 -> 0.00 mm
- net N$28: track 12.0 -> 0.00 mm
- net N$17: track 12.0 -> 0.00 mm
- net N$13: track 24.2 -> 13.4 mm
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
Commit message: update pcb design
Parts:
- added JP21: (no value), pinhead:1X01
- moved R4 1.00 mm to (17.3, 107.7)
- moved R3 0.50 mm to (27.3, 105.8)
Connections:
- net GND: now also JP21.1
Routing:
- net N$7: track 47.5 -> 48.5 mm
- net N$15: track 19.3 -> 18.3 mm
- net N$8: track 37.9 -> 37.4 mm
Changed lines of the file:
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@@
 <attribute name="VALUE" x="14.8" y="95.13" size="1.27" layer="28" rot="MR90"/>
 </element>
-<element name="R3" library="rcl" library_urn="urn:adsk.eagle:library:334" package="R1206" package3d_urn="urn:adsk.eagle:package:23540/2" value="220" x="27.34" y="106.32" smashed="yes" rot="MR90">
-<attribute name="NAME" x="28.61" y="105.05" size="1.27" layer="26" rot="MR90"/>
-<attribute name="POPULARITY" value="41" x="-46.32" y="149.5" size="1.778" layer="28" rot="MR90" display="off"/>
-<attribute name="SPICEPREFIX" value="R" x="-46.32" y="149.5" size="1.778" layer="28" rot="MR90" display="off"/>
-<attribute name="VALUE" x="24.8" y="105.05" size="1.27" layer="28" rot="MR90"/>
-</element>
-<element name="R4" library="rcl" library_urn="urn:adsk.eagle:library:334" package="R1206" package3d_urn="urn:adsk.eagle:package:23540/2" value="220" x="18.34" y="107.74" smashed="yes" rot="MR90">
-<attribute name="NAME" x="19.61" y="106.47" size="1.27" layer="26" rot="MR90"/>
-<attribute name="POPULARITY" value="41" x="-55.32" y="156" size="1.778" layer="28" rot="MR90" display="off"/>
-<attribute name="SPICEPREFIX" value="R" x="-55.32" y="156" size="1.778" layer="28" rot="MR90" display="off"/>
-<attribute name="VALUE" x="15.8" y="106.47" size="1.27" layer="28" rot="MR90"/>
+<element name="R3" library="rcl" library_urn="urn:adsk.eagle:library:334" package="R1206" package3d_urn="urn:adsk.eagle:package:23540/2" value="220" x="27.34" y="105.82" smashed="yes" rot="MR90">
+<attribute name="NAME" x="28.61" y="104.55" size="1.27" layer="26" rot="MR90"/>
+<attribute name="POPULARITY" value="41" x="-46.32" y="149" size="1.778" layer="28" rot="MR90" display="off"/>
+<attribute name="SPICEPREFIX" value="R" x="-46.32" y="149" size="1.778" layer="28" rot="MR90" display="off"/>
+<attribute name="VALUE" x="24.8" y="104.55" size="1.27" layer="28" rot="MR90"/>
+</element>
+<element name="R4" library="rcl" library_urn="urn:adsk.eagle:library:334" package="R1206" package3d_urn="urn:adsk.eagle:package:23540/2" value="220" x="17.34" y="107.74" smashed="yes" rot="MR90">
+<attribute name="NAME" x="18.61" y="106.47" size="1.27" layer="26" rot="MR90"/>
+<attribute name="POPULARITY" value="41" x="-56.32" y="156" size="1.778" layer="28" rot="MR90" display="off"/>
+<attribute name="SPICEPREFIX" value="R" x="-56.32" y="156" size="1.778" layer="28" rot="MR90" display="off"/>
+<attribute name="VALUE" x="14.8" y="106.47" size="1.27" layer="28" rot="MR90"/>
 </element>
 <element name="R5" library="rcl" library_urn="urn:adsk.eagle:library:334" package="R1206" package3d_urn="urn:adsk.eagle:package:23540/2" value="220" x="9.34" y="107.66" smashed="yes" rot="MR90">
@@
 <attribute name="POPULARITY" value="3" x="67" y="9.5" size="1.778" layer="27" display="off"/>
 <attribute name="VALUE" x="61.92" y="-0.025" size="1.778" layer="27" ratio="10"/>
+</element>
+<element name="JP21" library="pinhead" library_urn="urn:adsk.eagle:library:325" package="1X01" package3d_urn="urn:adsk.eagle:package:22485/2" value="" x="22" y="105.5" smashed="yes">
+<attribute name="NAME" x="20.6538" y="107.3288" size="1.27" layer="25" ratio="10"/>
+<attribute name="POPULARITY" value="64" x="22" y="105.5" size="1.778" layer="27" display="off"/>
+<attribute name="VALUE" x="20.73" y="102.325" size="1.27" layer="27"/>
 </element>
 </elements>
@@
 <wire x1="33.5" y1="96.5" x2="33.5" y2="109.5" width="0.6096" layer="16"/>
 <wire x1="33.5" y1="109.5" x2="32" y2="111" width="0.6096" layer="16"/>
-<wire x1="20.178" y1="111" x2="18.34" y2="109.162" width="0.6096" layer="16"/>
+<wire x1="19.178" y1="111" x2="17.34" y2="109.162" width="0.6096" layer="16"/>
 <wire x1="35.66" y1="94.34" x2="33.5" y2="96.5" width="0.6096" layer="16"/>
-<wire x1="32" y1="111" x2="20.178" y2="111" width="0.6096" layer="16"/>
+<wire x1="32" y1="111" x2="19.178" y2="111" width="0.6096" layer="16"/>
 </signal>
 <signal name="N$8">
@@
 <wire x1="38.23" y1="91.8" x2="34.2" y2="91.8" width="0.6096" layer="16"/>
 <wire x1="34.2" y1="91.8" x2="32" y2="94" width="0.6096" layer="16"/>
-<wire x1="32" y1="94" x2="32" y2="107.742" width="0.6096" layer="16"/>
-<wire x1="32" y1="107.742" x2="27.34" y2="107.742" width="0.6096" layer="16"/>
+<wire x1="32" y1="94" x2="32" y2="107.242" width="0.6096" layer="16"/>
+<wire x1="32" y1="107.242" x2="27.34" y2="107.242" width="0.6096" layer="16"/>
 </signal>
 <signal name="N$9">
@@
 <contactref element="BUS_B" pad="3"/>
 <contactref element="VBAT_B" pad="2"/>
+<contactref element="JP21" pad="1"/>
 </signal>
 <signal name="VCC">
@@
 <contactref element="LEDS" pad="3"/>
 <contactref element="R3" pad="1"/>
-<wire x1="27.34" y1="104.898" x2="25.84" y2="104.898" width="0.6096" layer="16"/>
-<wire x1="25.84" y1="104.898" x2="22.442" y2="101.5" width="0.6096" layer="16"/>
+<wire x1="27.34" y1="104.398" x2="25.34" y2="104.398" width="0.6096" layer="16"/>
+<wire x1="25.34" y1="104.398" x2="22.442" y2="101.5" width="0.6096" layer="16"/>
 <wire x1="22.442" y1="101.5" x2="16.5" y2="101.5" width="0.6096" layer="16"/>
 <wire x1="16.5" y1="101.5" x2="15" y2="100" width="0.6096" layer="16"/>
@@
 <contactref element="LEDS" pad="4"/>
 <contactref element="R4" pad="1"/>
-<wire x1="18.34" y1="106.318" x2="18.022" y2="106" width="0.6096" layer="16"/>
-<wire x1="18.022" y1="106" x2="15" y2="106" width="0.6096" layer="16"/>
+<wire x1="17.34" y1="106.318" x2="17.022" y2="106" width="0.6096" layer="16"/>
+<wire x1="17.022" y1="106" x2="15" y2="106" width="0.6096" layer="16"/>
 <wire x1="15" y1="106" x2="13" y2="104" width="0.6096" layer="16"/>
 <wire x1="13" y1="94.77" x2="9.2" y2="94.77" width="0.6096" layer="16"/>

Commit message: update ema pcb design
Parts:
- added JP22, JP23, JP24: (no value), pinhead:1X01
Connections:
- net GND: now also JP22.1, JP23.1, JP24.1
Routing:
- net VCC: track 333.3 -> 331.5 mm
Changed lines of the file:
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@@
 <attribute name="VALUE" x="20.73" y="102.325" size="1.27" layer="27"/>
+</element>
+<element name="JP22" library="pinhead" library_urn="urn:adsk.eagle:library:325" package="1X01" package3d_urn="urn:adsk.eagle:package:22485/2" value="" x="89" y="4.5" smashed="yes">
+<attribute name="NAME" x="87.6538" y="6.3288" size="1.27" layer="25" ratio="10"/>
+<attribute name="POPULARITY" value="64" x="89" y="4.5" size="1.778" layer="27" display="off"/>
+<attribute name="VALUE" x="87.73" y="1.325" size="1.27" layer="27"/>
+</element>
+<element name="JP23" library="pinhead" library_urn="urn:adsk.eagle:library:325" package="1X01" package3d_urn="urn:adsk.eagle:package:22485/2" value="" x="51.5" y="14" smashed="yes">
+<attribute name="NAME" x="50.1538" y="15.8288" size="1.27" layer="25" ratio="10"/>
+<attribute name="POPULARITY" value="64" x="51.5" y="14" size="1.778" layer="27" display="off"/>
+<attribute name="VALUE" x="50.23" y="10.825" size="1.27" layer="27"/>
+</element>
+<element name="JP24" library="pinhead" library_urn="urn:adsk.eagle:library:325" package="1X01" package3d_urn="urn:adsk.eagle:package:22485/2" value="" x="12.5" y="9" smashed="yes">
+<attribute name="NAME" x="11.1538" y="10.8288" size="1.27" layer="25" ratio="10"/>
+<attribute name="POPULARITY" value="64" x="12.5" y="9" size="1.778" layer="27" display="off"/>
+<attribute name="VALUE" x="11.23" y="5.825" size="1.27" layer="27"/>
 </element>
 </elements>
@@
 <contactref element="VBAT_B" pad="2"/>
 <contactref element="JP21" pad="1"/>
+<contactref element="JP22" pad="1"/>
+<contactref element="JP23" pad="1"/>
+<contactref element="JP24" pad="1"/>
 </signal>
 <signal name="VCC">
 <contactref element="BOARD1" pad="VIN"/>
 <contactref element="JP2" pad="15"/>
-<wire x1="59" y1="117" x2="107" y2="117" width="1.27" layer="1"/>
+<wire x1="59" y1="117" x2="102.5" y2="117" width="1.27" layer="1"/>
 <wire x1="59" y1="117" x2="55" y2="113" width="1.27" layer="1"/>
 <contactref element="R6" pad="2"/>
@@
 <contactref element="BUS" pad="4"/>
 <contactref element="DISPLAY" pad="3"/>
-<wire x1="107" y1="117" x2="112.51" y2="111.49" width="1.27" layer="1"/>
+<wire x1="112.5" y1="108.5" x2="111" y2="108.5" width="1.27" layer="1"/>
+<wire x1="111" y1="108.5" x2="102.5" y2="117" width="1.27" layer="1"/>
 <wire x1="112.51" y1="102.8" x2="112.51" y2="99.01" width="1.27" layer="16"/>
 <wire x1="112.51" y1="99.01" x2="109.97" y2="96.47" width="1.27" layer="16"/>
@@
 <wire x1="55" y1="74" x2="55" y2="21" width="1.27" layer="1"/>
 <wire x1="56" y1="74" x2="55" y2="74" width="1.27" layer="1"/>
-<wire x1="112.51" y1="111.49" x2="112.51" y2="108.51" width="1.27" layer="1"/>
-<wire x1="112.51" y1="108.51" x2="112.5" y2="108.5" width="1.27" layer="1"/>
 <wire x1="112.5" y1="108.5" x2="112.51" y2="108.49" width="1.27" layer="16"/>
 <wire x1="112.51" y1="108.49" x2="112.51" y2="102.8" width="1.27" layer="16"/>
