File: PCB_EMA/EMA_3/board.sch (EAGLE design)
At the start: 28 parts

Commit message: added PCBS and EAGLE filfes
Parts:
- added ., LORA: (no value), pinhead:PINHD-1X8
- added BUS_B: (no value), con-ptr500:AK500/4-H
- added JP10, JP11, JP12, JP13, JP14, JP15, JP16, JP17, JP18, JP19, JP20, JP4, JP5, JP6, JP7, JP8, JP9: (no value), pinhead:PINHD-1X1
- added VBAT_B: (no value), con-ptr500:AK500/2-H
- BUS: value RJ45-6L-B -> (none); device con-tycoelectronics:RJ45-6L-B -> pinhead:PINHD-1X4
- DISPLAY: device pinhead:PINHD-1X6 -> pinhead:PINHD-1X4
Connections:
- removed net N$12: BOARD1.D12, JP2.12
- removed net N$17: BOARD1.3V3, JP1.15
- removed net N$28: BOARD1.D15, JP1.13
- new net 3V3: ..3, BOARD1.3V3, JP1.15
- new net DIO0: ..5, BOARD1.D15, JP1.13
- new net DMISO: BOARD1.D12, JP2.12, LORA.4
- new net N$27: LORA.6
- new net N$29: LORA.7
- net DCS: now also JP13.1, JP14.1, LORA.2; no longer DISPLAY.6
- net DMOSI: now also LORA.3; no longer DISPLAY.4
- net DRST: now also ..4; no longer DISPLAY.5
- net DSCK: now also LORA.5; no longer DISPLAY.3
- net GND: now also ..1, ..2, BUS.3, BUS_B-3.KL, DISPLAY.4, JP15.1, JP16.1, JP17.1, JP18.1, JP19.1, JP20.1, LORA.1, LORA.8, VBAT_B-2.KL; no longer BUS.7, DISPLAY.1
- net MISO: now also JP11.1, JP12.1
- net SCL: now also BUS.2, BUS_B-2.KL, DISPLAY.2, JP10.1, JP9.1; no longer BUS.6
- net SDA: now also BUS.1, BUS_B-1.KL, DISPLAY.1, JP7.1, JP8.1; no longer BUS.5
- net VCC: now also BUS.4, BUS_B-4.KL, DISPLAY.3, JP4.1, JP5.1, JP6.1; no longer BUS.8, DISPLAY.2
- net VIN: now also VBAT_B-1.KL

Commit message: update pcb design
Parts:
- added JP21: (no value), pinhead:PINHD-1X1
Connections:
- net GND: now also JP21.1
Changed lines of the file:
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@@
 <part name="BUS_B" library="con-ptr500" library_urn="urn:adsk.eagle:library:181" deviceset="AK500/4-H" device="" package3d_urn="urn:adsk.eagle:package:9908/1"/>
 <part name="VBAT_B" library="con-ptr500" library_urn="urn:adsk.eagle:library:181" deviceset="AK500/2-H" device="" package3d_urn="urn:adsk.eagle:package:9901/1"/>
+<part name="JP21" library="pinhead" library_urn="urn:adsk.eagle:library:325" deviceset="PINHD-1X1" device="" package3d_urn="urn:adsk.eagle:package:22485/2"/>
 </parts>
 <sheets>
@@
 <attribute name="VALUE" x="3.81" y="-92.583" size="1.778" layer="96"/>
 </instance>
+<instance part="JP21" gate="G$1" x="213.36" y="-40.64" smashed="yes">
+<attribute name="NAME" x="207.01" y="-37.465" size="1.778" layer="95"/>
+<attribute name="VALUE" x="207.01" y="-45.72" size="1.778" layer="96"/>
+</instance>
 </instances>
 <busses>
@@
 <label x="17.78" y="-88.9" size="1.778" layer="95"/>
 </segment>
-</net>
+<segment>
+<pinref part="JP21" gate="G$1" pin="1"/>
+<wire x1="210.82" y1="-40.64" x2="203.2" y2="-40.64" width="0.1524" layer="91"/>
+<label x="203.2" y="-40.64" size="1.778" layer="95"/>
+</segment>
+</net>

Commit message: update ema pcb design
Parts:
- added JP22, JP23, JP24: (no value), pinhead:PINHD-1X1
Connections:
- net GND: now also JP22.1, JP23.1, JP24.1
Changed lines of the file:
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@@
 <part name="VBAT_B" library="con-ptr500" library_urn="urn:adsk.eagle:library:181" deviceset="AK500/2-H" device="" package3d_urn="urn:adsk.eagle:package:9901/1"/>
 <part name="JP21" library="pinhead" library_urn="urn:adsk.eagle:library:325" deviceset="PINHD-1X1" device="" package3d_urn="urn:adsk.eagle:package:22485/2"/>
+<part name="JP22" library="pinhead" library_urn="urn:adsk.eagle:library:325" deviceset="PINHD-1X1" device="" package3d_urn="urn:adsk.eagle:package:22485/2"/>
+<part name="JP23" library="pinhead" library_urn="urn:adsk.eagle:library:325" deviceset="PINHD-1X1" device="" package3d_urn="urn:adsk.eagle:package:22485/2"/>
+<part name="JP24" library="pinhead" library_urn="urn:adsk.eagle:library:325" deviceset="PINHD-1X1" device="" package3d_urn="urn:adsk.eagle:package:22485/2"/>
 </parts>
 <sheets>
@@
 <attribute name="VALUE" x="207.01" y="-45.72" size="1.778" layer="96"/>
 </instance>
+<instance part="JP22" gate="G$1" x="213.36" y="-53.34" smashed="yes">
+<attribute name="NAME" x="207.01" y="-50.165" size="1.778" layer="95"/>
+<attribute name="VALUE" x="207.01" y="-58.42" size="1.778" layer="96"/>
+</instance>
+<instance part="JP23" gate="G$1" x="226.06" y="-40.64" smashed="yes">
+<attribute name="NAME" x="219.71" y="-37.465" size="1.778" layer="95"/>
+<attribute name="VALUE" x="219.71" y="-45.72" size="1.778" layer="96"/>
+</instance>
+<instance part="JP24" gate="G$1" x="226.06" y="-53.34" smashed="yes">
+<attribute name="NAME" x="219.71" y="-50.165" size="1.778" layer="95"/>
+<attribute name="VALUE" x="219.71" y="-58.42" size="1.778" layer="96"/>
+</instance>
 </instances>
 <busses>
@@
 <label x="203.2" y="-40.64" size="1.778" layer="95"/>
 </segment>
-</net>
+<segment>
+<pinref part="JP22" gate="G$1" pin="1"/>
+<wire x1="210.82" y1="-53.34" x2="203.2" y2="-53.34" width="0.1524" layer="91"/>
+<label x="203.2" y="-53.34" size="1.778" layer="95"/>
+</segment>
+<segment>
+<pinref part="JP23" gate="G$1" pin="1"/>
+<wire x1="223.52" y1="-40.64" x2="218.44" y2="-40.64" width="0.1524" layer="91"/>
+<label x="215.9" y="-40.64" size="1.778" layer="95"/>
+</segment>
+<segment>
+<pinref part="JP24" gate="G$1" pin="1"/>
+<wire x1="223.52" y1="-53.34" x2="218.44" y2="-53.34" width="0.1524" layer="91"/>
+<label x="215.9" y="-53.34" size="1.778" layer="95"/>
+</segment>
+</net>
